Commit message: refactor: update package dependencies,  improve  configuration for gripper simulation, update to work with latest agx_arm_ros
- Changed maintainer email in package.xml
- Updated MoveIt package dependency from piper_with_gripper_moveit to agx_arm_moveit
- Enhanced launch file to streamline the integration of MoveIt and Gazebo
- Added support for gripper_joint2 in controller configurations
- Corrected URDF file references for accurate hardware description

File: urdf/piper_gzsim.ros2_control.xacro (robot description, xacro)
@@ -73,8 +73,9 @@
       </joint>
       <!--
-        gripper_joint2 is a mimic joint (multiplier=-1).
-        State-only: Gazebo handles the constraint from the <mimic> tag.
+        gripper_joint2 mirrors gripper_joint1 (multiplier=-1).
+        Commanded directly so MoveIt can dispatch trajectories for both joints.
       -->
       <joint name="gripper_joint2">
+        <command_interface name="position"/>
         <state_interface name="position">
           <param name="initial_value">${-1.0 * initial_positions['gripper_joint1']}</param>

File: urdf/piper_with_gripper_gzsim.urdf.xacro (robot description, xacro)
@@ -5,5 +5,5 @@
   <!-- Kinematics, visuals, collisions -->
   <xacro:include
-    filename="$(find agx_arm_description)/agx_arm_urdf/piper/urdf/piper_with_gripper_realsense_description.xacro"/>
+    filename="$(find agx_arm_description)/agx_arm_urdf/piper/urdf/piper_with_gripper_description.xacro"/>
   <!-- ros2_control hardware block (GazeboSimSystem) -->
   <xacro:include filename="$(find agx_arm_gzsim)/urdf/piper_gzsim.ros2_control.xacro"/>
